Commit message: second project robot model done

File: PR2/my_robot/urdf/my_robot.xacro (robot description, xacro)
@@ -29,4 +29,7 @@
         <cylinder radius="0.2" length="0.1"/>
       </geometry>
+      <material name="chassis_color">
+        <color rgba="0.5 0.5 0.5 1.0"/> <!-- Gray color -->
+      </material>
     </visual>
   </link>
@@ -51,4 +54,7 @@
         <sphere radius="0.05"/>
       </geometry>
+      <material name="caster_color">
+        <color rgba="0.8 0.2 0.2 1.0"/> <!-- Red color -->
+      </material>
     </visual>
   </link>
@@ -57,4 +63,72 @@
     <parent link="chassis"/>
     <child link="front_caster"/>
+  </joint>
+   <!-- Camera Link -->
+  <link name="camera">
+    <inertial>
+      <mass value="0.1"/>
+      <origin xyz="0 0 0" rpy="0 0 0"/>
+      <inertia
+          ixx="1e-6" ixy="0" ixz="0"
+          iyy="1e-6" iyz="0"
+          izz="1e-6"
+      />
+    </inertial>
+    <collision>
+      <origin xyz="0 0 0" rpy="0 0 0"/>
+      <geometry>
+        <box size="0.05 0.05 0.05"/>
+      </geometry>
+    </collision>
+    <visual>
+      <origin xyz="0 0 0" rpy="0 0 0"/>
+      <geometry>
+        <box size="0.05 0.05 0.05"/>
+      </geometry>
+      <material name="camera_color">
+        <color rgba="0.2 0.8 0.2 1.0"/> <!-- Green color -->
+      </material>
+    </visual>
+  </link>
+  <!-- Camera Joint -->
+  <joint name="camera_joint" type="fixed">
+    <origin xyz="0.2 0 0" rpy="0 0 0"/>
+    <parent link="chassis"/>
+    <child link="camera"/>
+    <axis xyz="0 1 0"/>
+  </joint>
+   <!-- Hokuyo Link -->
+  <link name="hokuyo">
+    <inertial>
+      <mass value="1e-5"/>
+      <origin xyz="0 0 0" rpy="0 0 0"/>
+      <inertia
+          ixx="1e-6" ixy="0" ixz="0"
+          iyy="1e-6" iyz="0"
+          izz="1e-6"
+      />
+    </inertial>
+    <collision>
+      <origin xyz="0 0 0" rpy="0 0 0"/>
+      <geometry>
+        <box size="0.1 0.1 0.1"/>
+      </geometry>
+    </collision>
+    <visual>
+      <origin xyz="0 0 0" rpy="0 0 0"/>
+      <geometry>
+        <mesh filename="package://my_robot/meshes/hokuyo.dae"/>
+      </geometry>
+      <material name="hokuyo_color">
+        <color rgba="0.2 0.2 0.2 1.0"/> <!-- Dark Gray -->
+      </material>
+    </visual>
+  </link>
+  <!-- Hokuyo Joint -->
+  <joint name="hokuyo_joint" type="fixed">
+    <origin xyz="0.15 0 0.085" rpy="0 0 0"/>
+    <parent link="chassis"/>
+    <child link="hokuyo"/>
+    <axis xyz="0 1 0"/>
   </joint>
   <!-- Left Wheel -->
@@ -80,4 +154,7 @@
         <cylinder radius="0.08" length="0.02"/>
       </geometry>
+      <material name="wheel_color">
+        <color rgba="0.2 0.2 0.8 1.0"/> <!-- Blue color -->
+      </material>
     </visual>
   </link>
@@ -112,7 +189,4 @@
         <cylinder radius="0.08" length="0.02"/>
       </geometry>
-      <material name="">
-        <color rgba="0.75294 0.75294 0.75294 1"/>
-      </material>
     </visual>
   </link>
@@ -125,3 +199,18 @@
     <dynamics damping="1.0" friction="1.0"/>
   </joint>
+  <gazebo reference="chassis">
+	<material>Gazebo/Blue</material>
+  </gazebo>
+  <gazebo reference="camera">
+	<material>Gazebo/Red</material>
+  </gazebo>
+  <gazebo reference="left_wheel">
+	<material>Gazebo/Green</material>
+   </gazebo>
+   <gazebo reference="right_wheel">
+	<material>Gazebo/Green</material>
+   </gazebo>
+   <gazebo reference="front_caster">
+	<material>Gazebo/Yellow</material>
+   </gazebo>
 </robot>

Commit message: pub and serv complete

File: PR2/my_robot/urdf/my_robot.xacro (robot description, xacro)
@@ -1,4 +1,5 @@
 <?xml version='1.0'?>
 <robot name="my_robot" xmlns:xacro="http://www.ros.org/wiki/xacro">
+<xacro:include filename="$(find my_robot)/urdf/my_robot.gazebo" />
   <link name="robot_footprint"></link>
   <joint name="robot_footprint_joint" type="fixed">
@@ -21,5 +22,5 @@
       <origin xyz="0 0 0" rpy=" 0 0 0"/>
       <geometry>
-        <cylinder radius="0.2" length="0.1"/>
+        <cylinder radius="0.17" length="0.12"/>
       </geometry>
     </collision>
@@ -27,41 +28,32 @@
       <origin xyz="0 0 0" rpy=" 0 0 0"/>
       <geometry>
-        <cylinder radius="0.2" length="0.1"/>
-      </geometry>
-      <material name="chassis_color">
-        <color rgba="0.5 0.5 0.5 1.0"/> <!-- Gray color -->
-      </material>
-    </visual>
-  </link>
-  <!-- Front Caster -->
-  <link name="front_caster">
-    <inertial>
-      <mass value="0.5"/>
-      <origin xyz="0 0 0" rpy="0 0 0"/>
-      <inertia
-          ixx="0.01" ixy="0" ixz="0"
-          iyy="0.01" iyz="0"
-          izz="0.01"
-      />
-    </inertial>
-    <collision>
+        <cylinder radius="0.17" length="0.12"/>
+      </geometry>
+    </visual>
+  <collision name='back_caster_collision'>
+      <origin xyz="-0.12 0 -0.05" rpy=" 0 0 0"/>
+      <geometry>
+        <sphere radius="0.0499"/>
+      </geometry>
+    </collision>
+    <visual name='back_caster_visual'>
+      <origin xyz="-0.12 0 -0.05" rpy=" 0 0 0"/>
       <geometry>
         <sphere radius="0.05"/>
       </geometry>
-    </collision>
-    <visual>
+    </visual>
+    <collision name='front_caster_collision'>
+      <origin xyz="0.12 0 -0.05" rpy=" 0 0 0"/>
+      <geometry>
+        <sphere radius="0.0499"/>
+      </geometry>
+    </collision>
+    <visual name='front_caster_visual'>
+      <origin xyz="0.12 0 -0.05" rpy=" 0 0 0"/>
       <geometry>
         <sphere radius="0.05"/>
       </geometry>
-      <material name="caster_color">
-        <color rgba="0.8 0.2 0.2 1.0"/> <!-- Red color -->
-      </material>
-    </visual>
-  </link>
-  <joint name="front_caster_joint" type="fixed">
-    <origin xyz="0.15 0 -0.05" rpy="0 0 0"/>
-    <parent link="chassis"/>
-    <child link="front_caster"/>
-  </joint>
+    </visual>
+  </link>
    <!-- Camera Link -->
   <link name="camera">
@@ -127,5 +119,5 @@
   <!-- Hokuyo Joint -->
   <joint name="hokuyo_joint" type="fixed">
-    <origin xyz="0.15 0 0.085" rpy="0 0 0"/>
+    <origin xyz="0.15 0 0.1" rpy="0 0 0"/>
     <parent link="chassis"/>
     <child link="hokuyo"/>
@@ -135,30 +127,25 @@
   <link name="left_wheel">
     <inertial>
-      <mass value="0.5"/>
-      <origin xyz="0 0 0" rpy="0 0 0"/>
-      <inertia
-          ixx="0.02" ixy="0" ixz="0"
-          iyy="0.02" iyz="0"
-          izz="0.03"
-      />
-    </inertial>
-    <collision>
-      <origin xyz="0 0 0" rpy="1.5707 0 0"/>
-      <geometry>
-        <cylinder radius="0.08" length="0.02"/>
-      </geometry>
-    </collision>
-    <visual>
-      <origin xyz="0 0 0" rpy="1.5707 0 0"/>
-      <geometry>
-        <cylinder radius="0.08" length="0.02"/>
-      </geometry>
-      <material name="wheel_color">
-        <color rgba="0.2 0.2 0.8 1.0"/> <!-- Blue color -->
-      </material>
+      <mass value="5"/>
+      <origin xyz="0 0 0" rpy="0 1.5707 1.5707"/>
+      <inertia
+         ixx="0.1" ixy="0" ixz="0" iyy="0.1" iyz="0" izz="0.1"
+      />
+    </inertial>
+    <collision>
+      <origin xyz="0 0 0" rpy="0 1.5707 1.5707"/>
+      <geometry>
+        <cylinder radius="0.1" length="0.05"/>
+      </geometry>
+    </collision>
+    <visual>
+      <origin xyz="0 0 0" rpy="0 1.5707 1.5707"/>
+      <geometry>
+        <cylinder radius="0.1" length="0.05"/>
+      </geometry>
     </visual>
   </link>
   <joint type="continuous" name="left_wheel_joint">
-    <origin xyz="-0.1 -0.2 0" rpy="0 0 0"/> <!-- Pinned to chassis edge -->
+    <origin xyz="0 0.15 0" rpy="0 0 0"/> <!-- Pinned to chassis edge -->
     <child link="left_wheel"/>
     <parent link="chassis"/>
@@ -170,27 +157,25 @@
   <link name="right_wheel">
     <inertial>
-      <mass value="0.5"/>
-      <origin xyz="0 0 0" rpy="0 0 0"/>
-      <inertia
-          ixx="0.02" ixy="0" ixz="0"
-          iyy="0.02" iyz="0"
-          izz="0.03"
-      />
-    </inertial>
-    <collision>
-      <origin xyz="0 0 0" rpy="1.5707 0 0"/>
-      <geometry>
-        <cylinder radius="0.08" length="0.02"/>
-      </geometry>
-    </collision>
-    <visual>
-      <origin xyz="0 0 0" rpy="1.5707 0 0"/>
-      <geometry>
-        <cylinder radius="0.08" length="0.02"/>
+      <mass value="5"/>
+      <origin xyz="0 0 0" rpy="0 1.5707 1.5707"/>
+      <inertia
+         ixx="0.1" ixy="0" ixz="0" iyy="0.1" iyz="0" izz="0.1"
+      />
+    </inertial>
+    <collision>
+      <origin xyz="0 0 0" rpy="0 1.5707 1.5707"/>
+      <geometry>
+        <cylinder radius="0.1" length="0.05"/>
+      </geometry>
+    </collision>
+    <visual>
+      <origin xyz="0 0 0" rpy="0 1.5707 1.5707"/>
+      <geometry>
+        <cylinder radius="0.1" length="0.05"/>
       </geometry>
     </visual>
   </link>
   <joint type="continuous" name="right_wheel_joint">
-    <origin xyz="-0.1 0.2 0" rpy="0 0 0"/> <!-- Pinned to chassis edge -->
+    <origin xyz="0 -0.15 0" rpy="0 0 0"/> <!-- Pinned to chassis edge -->
     <child link="right_wheel"/>
     <parent link="chassis"/>
@@ -211,6 +196,9 @@
 	<material>Gazebo/Green</material>
    </gazebo>
-   <gazebo reference="front_caster">
+   <gazebo reference="back_caster_visual">
 	<material>Gazebo/Yellow</material>
    </gazebo>
+     <gazebo reference="front_caster_visual">
+	<material>Gazebo/Yellow</material>
+   </gazebo>
 </robot>
